Commit message: Nexus with camera, sonar and lidar

File: Nexus_Modified_Tommi/nexus_4wd_mecanum_simulator-master/nexus_4wd_mecanum_description/urdf/old/nexus_4wd_mecanum.xacro (robot description, xacro)
@@ -4,8 +4,4 @@
   <xacro:property name="wheel_radius" value="0.050" />
   <xacro:property name="wheel_width" value="0.0505" />
-  <!-- Determine presence of Hokuyo laser sensor -->
-  <xacro:arg name="add_laser_sensor" default="true" />
-  <!-- Determine presence of RGB camera sensor -->
-  <xacro:arg name="add_camera_sensor" default="true" />
   <material name="yellow"><color rgba="0.8 0.8 0.0 1.0" /></material>
   <material name="black"><color rgba="0.15 0.15 0.15 1.0" /></material>
@@ -331,18 +327,125 @@
     </visual>
   </link>
-  <!-- Add a Hokuyo laser scanner -->
-  <xacro:if value="$(arg add_laser_sensor)">
-    <!-- Add Laser link, joints and mesh -->
-    <xacro:include filename="$(find nexus_4wd_mecanum_description)/urdf/hokuyo_laser.xacro"/>
-    <!-- Add Gazebo Laser Plugin -->
-    <xacro:include filename="$(find nexus_4wd_mecanum_description)/urdf/hokuyo_laser.gazebo"/>
-  </xacro:if>
-  <!-- Add a regular RGB Camera -->
-  <xacro:if value="$(arg add_camera_sensor)">
-    <!-- Add Camera link, joints and mesh -->
-    <xacro:include filename="$(find nexus_4wd_mecanum_description)/urdf/rgb_camera.xacro"/>
-    <!-- Add Gazebo Camera Plugin -->
-    <xacro:include filename="$(find nexus_4wd_mecanum_description)/urdf/rgb_camera.gazebo"/>
-  </xacro:if>
+  <!--LIDAR-->
+  <!-- TENTATIVO 1: NON LEGGE MSG
+  <link name="lidar_link">
+    <inertial>
+      <origin xyz="0 0 0" rpy="0 0 0"/>
+      <mass value="0.125"/>
+      <inertia ixx="0.001"  ixy="0"  ixz="0" iyy="0.001" iyz="0" izz="0.001" />
+    </inertial>
+    <collision>
+      <origin xyz="0 0 0" rpy="0 0 0"/>
+      <geometry>
+         <cylinder radius="0.0508" length="0.055"/>
+      </geometry>
+    </collision>
+    <visual>
+      <origin xyz="0 0 0" rpy="0 0 0"/>
+      <geometry>
+         <cylinder radius="0.0508" length="0.055"/>
+      </geometry>
+    </visual>
+  </link>
+  <joint name="lidar_joint" type="fixed">
+    <parent link="base_link"/>
+    <child link="lidar_link"/>
+    <origin xyz="0 0 0.055" rpy="0 0 0"/>
+  </joint>
+  <gazebo reference="lidar_link">
+    <sensor name="lidar" type="ray">
+      <always_on>true</always_on>
+      <visualize>true</visualize>
+      <update_rate>5</update_rate>
+      <ray>
+        <scan>
+          <horizontal>
+            <samples>360</samples>
+            <resolution>1.000000</resolution>
+            <min_angle>0.000000</min_angle>
+            <max_angle>6.280000</max_angle>
+          </horizontal>
+        </scan>
+        <range>
+          <min>0.120000</min>
+          <max>3.5</max>
+          <resolution>0.015000</resolution>
+        </range>
+        <noise>
+          <type>gaussian</type>
+          <mean>0.0</mean>
+          <stddev>0.01</stddev>
+        </noise>
+      </ray>
+      <plugin name="gazebo_ros_head_hokuyo_controlle" filename="libgazebo_ros_ray_sensor.so" >
+        <ros>
+          <remapping>~/out:=/scan</remapping>
+        </ros>
+        <output_type>sensor_msgs/LaserScan</output_type>
+      </plugin>
+  </gazebo>
+  -->
+  <!--TENTATIVO 2: hoyuko, from http://gazebosim.org/tutorials?tut=ros_gzplugins#Laser-->
+  <!--
+  <joint name="hokuyo_joint" type="fixed">
+    <origin xyz="0 0 0.055" rpy="0 0 0"/>
+    <parent link="base_link"/>
+    <child link="hokuyo_link"/>
+  </joint>
+  <link name="hokuyo_link">
+    <collision>
+      <origin xyz="0 0 0" rpy="0 0 0"/>
+      <geometry>
+    <box size="0.1 0.1 0.1"/>
+      </geometry>
+    </collision>
+    <visual>
+      <origin xyz="0 0 0" rpy="0 0 0"/>
+      <geometry>
+        <mesh filename="package://nexus_4wd_mecanum_description/meshes/hokuyo.dae"/>
+      </geometry>
+    </visual>
+    <inertial>
+      <mass value="1e-5" />
+      <origin xyz="0 0 0" rpy="0 0 0"/>
+      <inertia ixx="1e-6" ixy="0" ixz="0" iyy="1e-6" iyz="0" izz="1e-6" />
+    </inertial>
+  </link> -->
+ <!--TENTATIVO 3: hoyuko, from https://bitbucket.org/kiranpalla/learn-ros/src/8f5207d8e52c/using-gazebo-laser-scan/src/mybot/urdf/mybot.xacro-->
+  <xacro:include filename="$(find nexus_4wd_mecanum_description)/urdf/lidar_sensor.plugin.xacro" />
+  <xacro:property name="laser_size_x" value="0.03"/>
+  <xacro:property name="laser_size_y" value="0.03"/>
+  <xacro:property name="laser_size_z" value="0.04"/>
+  <xacro:property name="laser_origin_x" value="0.065"/>
+  <xacro:property name="laser_origin_y" value="0"/>
+  <xacro:property name="laser_origin_z" value="0.06"/>
+  <xacro:macro name="default_inertial" params="mass">
+    <inertial>
+      <mass value="${mass}"/>
+      <inertia ixx="1.0" ixy="0.0" ixz="0.0" iyy="1.0" iyz="0.0" izz="1.0"/>
+    </inertial>
+  </xacro:macro>
+  <!--Laser Scan-->
+  <link name="sensor_laser">
+    <visual>
+      <geometry>
+        <mesh filename="package://nexus_4wd_mecanum_description/meshes/hokuyo.dae"/>
+        <!--box size="${laser_size_x} ${laser_size_y} ${laser_size_z}"/-->
+      </geometry>
+      <material name="blue"/>
+    </visual>
+    <collision>
+      <geometry>
+        <box size="${laser_size_x} ${laser_size_y} ${laser_size_z}"/>
+      </geometry>
+    </collision>
+    <xacro:default_inertial mass="0.02"/>
+  </link>
+  <joint name="sensor_laser_joint" type="fixed">
+    <origin xyz="${laser_origin_x} ${laser_origin_y} ${laser_origin_z}" rpy="0 0 0" />
+    <parent link="base_link"/>
+    <child link="sensor_laser" />
+  </joint>
+  <!--FINE LIDAR-->
   <!-- Include controller plugin for Gazebo -->
   <xacro:include filename="$(find nexus_4wd_mecanum_description)/urdf/nexus_4wd_mecanum.gazebo" />
